Commit message: main

File: Project2/Project2/src/my_robot/urdf/my_robot.xacro (robot description, xacro)
@@ -43,4 +43,5 @@
       </geometry>
     </visual>
+<!--
     <collision name='front_caster_collision'>
       <origin xyz="0.15 0 -0.05" rpy=" 0 0 0"/>
@@ -55,4 +56,5 @@
       </geometry>
     </visual>
+ -->
   </link>
   <link name='left_wheel'>
@@ -79,4 +81,12 @@
     </visual>
   </link>
+  <joint type="continuous" name="left_wheel_hinge">
+    <origin xyz="0 0.15 0" rpy="0 0 0"/>
+    <child link="left_wheel"/>
+    <parent link="chassis"/>
+    <axis xyz="0 1 0" rpy="0 0 0"/>
+    <limit effort="10000" velocity="1000"/>
+    <dynamics damping="1.0" friction="1.0"/>
+  </joint>
   <link name='right_wheel'>
     <inertial>
@@ -102,12 +112,4 @@
     </visual>
   </link>
-  <joint type="continuous" name="left_wheel_hinge">
-    <origin xyz="0 0.15 0" rpy="0 0 0"/>
-    <child link="left_wheel"/>
-    <parent link="chassis"/>
-    <axis xyz="0 1 0" rpy="0 0 0"/>
-    <limit effort="10000" velocity="1000"/>
-    <dynamics damping="1.0" friction="1.0"/>
-  </joint>
   <joint type="continuous" name="right_wheel_hinge">
     <origin xyz="0 -0.15 0" rpy="0 0 0"/>
@@ -118,4 +120,124 @@
     <dynamics damping="1.0" friction="1.0"/>
   </joint>
+  <link name='top1'>
+    <pose>0 0 0.1 0 0 0</pose>
+    <inertial>
+      <mass value="0.1"/>
+      <origin xyz="0.0 0 0" rpy=" 0 0 0"/>
+      <inertia
+          ixx="1e-6" ixy="0" ixz="0"
+          iyy="1e-6" iyz="0"
+          izz="1e-6"
+      />
+    </inertial>
+    <collision name='collision'>
+      <origin xyz="0 0 0" rpy=" 0 0 0"/>
+      <geometry>
+        <box size=".4 .2 .1"/>
+      </geometry>
+    </collision>
+    <visual name='top1_visual'>
+      <origin xyz="0 0 0" rpy=" 0 0 0"/>
+      <geometry>
+        <box size=".4 .2 .1"/>
+      </geometry>
+    </visual>
+  </link>
+  <joint type="fixed" name="top1_joint">
+    <origin xyz="0 0 0.098" rpy="0 0 0"/>
+    <child link="top1"/>
+    <parent link="chassis"/>
+    <axis xyz="0 1 0" rpy="0 0 0"/>
+  </joint>
+  <link name='top_cylinder'>
+    <pose>0 0 0.1 0 0 0</pose>
+    <inertial>
+      <mass value="0.1"/>
+      <origin xyz="0.0 0 0" rpy=" 0 0 0"/>
+      <inertia
+          ixx="1e-6" ixy="0" ixz="0"
+          iyy="1e-6" iyz="0"
+          izz="1e-6"
+      />
+    </inertial>
+    <collision name='collision'>
+      <origin xyz="0 0 0" rpy=" 0 0 0"/>
+      <geometry>
+        <cylinder radius='.25' length='.05'/>
+      </geometry>
+    </collision>
+    <visual name='top_cylinder_visual'>
+      <origin xyz="0 0 0" rpy=" 0 0 0"/>
+      <geometry>
+        <cylinder radius='.25' length='.05'/>
+      </geometry>
+    </visual>
+  </link>
+  <joint type="fixed" name="top_cylinder_joint">
+    <origin xyz="0 0 0.125" rpy="0 0 0"/>
+    <child link="top_cylinder"/>
+    <parent link="chassis"/>
+    <axis xyz="0 1 0" rpy="0 0 0"/>
+  </joint>
+  <link name='front_beam'>
+    <pose>0 0 0.1 0 0 0</pose>
+    <inertial>
+      <mass value="0.1"/>
+      <origin xyz="0.0 0 0" rpy=" 0 0 0"/>
+      <inertia
+          ixx="1e-6" ixy="0" ixz="0"
+          iyy="1e-6" iyz="0"
+          izz="1e-6"
+      />
+    </inertial>
+     <collision name='collision'>
+      <origin xyz="0 0 0" rpy=" 0 0 0"/>
+      <geometry>
+        <box size=".1 .2 .1"/>
+      </geometry>
+    </collision>
+    <visual name='front_beam_visual'>
+      <origin xyz="0 0 0" rpy=" 0 0 0"/>
+      <geometry>
+        <box size=".1 .2 .1"/>
+      </geometry>
+    </visual>
+  </link>
+  <joint type="fixed" name="front_beam_joint">
+    <origin xyz="0.15 0 -0.05" rpy="0 0 0"/>
+    <child link="front_beam"/>
+    <parent link="chassis"/>
+    <axis xyz="0 1 0" rpy="0 0 0"/>
+  </joint>
+  <link name='front_wiper'>
+    <pose>0 0 0.1 0 0 0</pose>
+    <inertial>
+      <mass value="0.1"/>
+      <origin xyz="0.0 0 0" rpy=" 0 0 0"/>
+      <inertia
+          ixx="1e-6" ixy="0" ixz="0"
+          iyy="1e-6" iyz="0"
+          izz="1e-6"
+      />
+    </inertial>
+     <collision name='collision'>
+      <origin xyz="0 0 0" rpy=" 0 0 0"/>
+      <geometry>
+        <box size=".155 .4 .025"/>
+      </geometry>
+    </collision>
+    <visual name='front_wiper_visual'>
+      <origin xyz="0 0 0" rpy=" 0 0 0"/>
+      <geometry>
+        <box size=".149 .4 .025"/>
+      </geometry>
+    </visual>
+  </link>
+  <joint type="fixed" name="front_wiper_joint">
+    <origin xyz="0.175 0 -0.0875" rpy="0 0 0"/>
+    <child link="front_wiper"/>
+    <parent link="chassis"/>
+    <axis xyz="0 1 0" rpy="0 0 0"/>
+  </joint>
   <link name='camera'>
     <inertial>
@@ -142,5 +264,5 @@
   </link>
   <joint type="fixed" name="camera_joint">
-    <origin xyz="0.2 0 0" rpy="0 0 0"/>
+    <origin xyz="0.2 0 0.05" rpy="0 0 0"/>
     <child link="camera"/>
     <parent link="chassis"/>
@@ -171,17 +293,29 @@
   </link>
   <joint type="fixed" name="hokuyo_joint">
-    <origin xyz="0.15 0 0.1" rpy="0 0 0"/>
+    <origin xyz="0.15 0 0.175" rpy="0 0 0"/>
     <child link="hokuyo"/>
     <parent link="chassis"/>
     <axis xyz="0 1 0" rpy="0 0 0"/>
   </joint>
+  <gazebo reference="chassis">
+    <material>Gazebo/Purple</material>
+  </gazebo>
   <gazebo reference="left_wheel">
+    <material>Gazebo/Black</material>
+  </gazebo>
+  <gazebo reference="right_wheel">
+    <material>Gazebo/Black</material>
+  </gazebo>
+  <gazebo reference="top_cylinder">
     <material>Gazebo/Green</material>
   </gazebo>
-  <gazebo reference="right_wheel">
-    <material>Gazebo/Green</material>
-  </gazebo>
-  <gazebo reference="chassis">
-    <material>Gazebo/Blue</material>
+  <gazebo reference="top1">
+    <material>Gazebo/Purple</material>
+  </gazebo>
+  <gazebo reference="front_beam">
+    <material>Gazebo/Purple</material>
+  </gazebo>
+  <gazebo reference="front_wiper">
+    <material>Gazebo/Orange</material>
   </gazebo>
   <gazebo reference="camera">
